File: rileyu0board.kicad_sch (KiCad schematic)
At the start: 1 part, among them IC1 STM32U073KCU3

Commit message: everything is wrong but stuff is happening
Parts:
- added J1: USB_C_Receptacle_USB2.0_16P, Riley:GCT_USB4520-03-0-A_REVA, symbol Connector:USB_C_Receptacle_USB2.0_16P
- added J2: Conn_01x12_Pin, Connector_JST:JST_PH_B12B-PH-SM4-TB_1x12-1MP_P2.00mm_Vertical, symbol Connector:Conn_01x12_Pin
- added J3: Conn_01x12_Pin, symbol Connector:Conn_01x12_Pin
- added SW1: SW_Nidec_CAS-120A1, Button_Switch_SMD:Nidec_Copal_CAS-120A, symbol Switch:SW_Nidec_CAS-120A1
- added X1: SG-3030CM, Oscillator:Oscillator_SMD_SeikoEpson_SG3030CM, symbol Oscillator:SG-3030CM
Connections:
- net +3V3: now reaches IC1.1 (VDD)
- net +3V3: now also SW1.1 (C)
- net at IC1.10 (PA4): now also J3.5 (Pin_5)
- net at IC1.11 (PA5): now also J3.6 (Pin_6)
- net at IC1.12 (PA6): now also J3.7 (Pin_7)
- net at IC1.13 (PA7): now also J3.8 (Pin_8)
- net at IC1.14 (PB0): now also J3.9 (Pin_9)
- net at IC1.15 (PB1): now also J3.10 (Pin_10)
- net GND: now reaches IC1.16 (VSS_1)
- net GND: now also IC1.32 (VSS_2), IC1.33 (EP), J1.A1 (GND), J1.A12 (GND), J1.B1 (GND), J1.B12 (GND), SW1.3 (A), X1.2 (GND)
- net at IC1.17 (VDDUSB): now also J1.A4 (VBUS), J1.A9 (VBUS), J1.B4 (VBUS), J1.B9 (VBUS)
- net at IC1.18 (PA8): now also J3.11 (Pin_11)
- net at IC1.19 (PA9): now also J3.12 (Pin_12)
- net at IC1.2 (PC14-OSC32_IN): now also X1.4 (Vcc)
- net at IC1.20 (PA10): now also J2.1 (Pin_1)
- net at IC1.21 (PA11_[PA9]): now also J2.2 (Pin_2)
- net at IC1.22 (PA12_[PA10]): now also J2.3 (Pin_3)
- net at IC1.23 (PA13): now also J2.4 (Pin_4)
- net at IC1.24 (PA14): now also J2.5 (Pin_5)
- net at IC1.25 (PA15): now also J2.6 (Pin_6)
- net at IC1.26 (PB3): now also J2.7 (Pin_7)
- net at IC1.27 (PB4): now also J2.8 (Pin_8)
- net at IC1.28 (PB5): now also J2.9 (Pin_9)
- net at IC1.29 (PB6): now also J2.10 (Pin_10)
- net at IC1.3 (PC15-OSC32_OUT): now also X1.1 (VIO)
- net at IC1.30 (PB7): now also J2.11 (Pin_11)
- net at IC1.31 (PF3-BOOT0): now also J2.12 (Pin_12)
- net at IC1.4 (PF2-NRST): now also SW1.2 (B)
- net +3.3VA: now reaches IC1.5 (VDDA/VREF+)
- net at IC1.6 (PA0-CK_IN): now also J3.1 (Pin_1)
- net at IC1.7 (PA1): now also J3.2 (Pin_2)
- net at IC1.8 (PA2): now also J3.3 (Pin_3)
- net at IC1.9 (PA3): now also J3.4 (Pin_4)
- no-connect marks 0 -> 10
